File: lasagna-motherboard/_autosave-lasagna-motherboard.kicad_pcb (KiCad board)
At the start: 2 copper layers, 230.4 x 97.8 mm, 16 parts, among them J1 Jetson_Power_Connector, J2 Fathom_X_Connector, J3 Power_Connector, U1 Adafruit_BNO055_IMU, U10 ESC, U11 ESC, U12 ESC, U13 ESC, U2 Jetson_Xavier_NX_Mounting_Hol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, U3 Jetson_Xavier_NX_Pins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

Commit message: created something
Parts:
- J1, U11, U12, U6, U8: moved to B.Cu
- moved J3 212.1 mm to (42.2, 112.8), turned to 90 degrees
- moved J2 211.1 mm to (41.4, 67.3), turned to 90 degrees
- moved J1 175.6 mm to (243.3, 149.6), turned to -90 degrees
- moved U6 106.4 mm to (143.8, 147.3), turned to 90 degrees
- moved U7 102.0 mm to (143.8, 84.8), turned to -90 degrees
- moved U9 96.6 mm to (125.7, 147.3), turned to -90 degrees
- moved U10 93.3 mm to (143.8, 126.2), turned to -90 degrees
- moved U12 86.4 mm to (126.0, 126.5), turned to 90 degrees
- moved U8 75.0 mm to (143.8, 104.6), turned to 90 degrees
- moved U13 57.5 mm to (126.0, 105.4), turned to -90 degrees
- moved U3 50.8 mm to (147.3, 70.1), turned to 180 degrees
- moved U11 47.5 mm to (126.0, 85.1), turned to 90 degrees
Other:
- outline, holes or cut-outs redrawn
