File: lasagna-motherboard/_autosave-lasagna-motherboard.kicad_sch (KiCad schematic)
At the start: 16 parts, among them J1 Jetson_Power_Connector, J2 Fathom_X_Connector, J3 Power_Connector, U1 Adafruit_BNO055_IMU, U10 ESC, U11 ESC, U12 ESC, U13 ESC, U2 Jetson_Xavier_NX_Mounting_Hol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, U3 Jetson_Xavier_NX_Pins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

Commit message: finished the schematic + created jetson power connector footprint
Parts:
- J1: footprint (none) -> lasagna-motherboard:Jetson Power Connector
- J2: footprint (none) -> lasagna-motherboard:FathomX_Connector
- J3: footprint (none) -> lasagna-motherboard:Power_Connector
- U1: footprint (none) -> lasagna-motherboard:Adafruit_BNO055_IMU
- U10, U11, U12, U13, U6, U7, U8, U9: footprint (none) -> lasagna-motherboard:ESC
- U2: footprint (none) -> lasagna-motherboard:Jetson_Xavier_NX_Mounting_Holes
- U3: footprint (none) -> lasagna-motherboard:Jetson_Xavier_NX_2X20_Pin_Header
- U4: footprint (none) -> lasagna-motherboard:FathomX
- U5: footprint (none) -> lasagna-motherboard:Adafruit_PCA9685_PWMGen
Changed lines of the file:
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@@
     (property "Reference" "U10" (id 0) (at 239.395 104.14 0))
     (property "Value" "ESC" (id 1) (at 239.395 106.68 0))
-    (property "Footprint" "" (id 2) (at 238.76 111.76 0)
+    (property "Footprint" "lasagna-motherboard:ESC" (id 2) (at 238.76 111.76 0)
       (effects (font (size 1.27 1.27)) hide)
     )
@@
     (property "Reference" "U8" (id 0) (at 239.395 73.66 0))
     (property "Value" "ESC" (id 1) (at 239.395 76.2 0))
-    (property "Footprint" "" (id 2) (at 238.76 81.28 0)
+    (property "Footprint" "lasagna-motherboard:ESC" (id 2) (at 238.76 81.28 0)
       (effects (font (size 1.27 1.27)) hide)
     )
@@
       (effects (font (size 1.27 1.27)) (justify left))
     )
-    (property "Footprint" "" (id 2) (at 104.14 34.29 0)
+    (property "Footprint" "lasagna-motherboard:Jetson_Xavier_NX_Mounting_Holes" (id 2) (at 104.14 34.29 0)
       (effects (font (size 1.27 1.27)) hide)
     )
@@
     (property "Reference" "U12" (id 0) (at 239.395 130.81 0))
     (property "Value" "ESC" (id 1) (at 239.395 133.35 0))
-    (property "Footprint" "" (id 2) (at 238.76 138.43 0)
+    (property "Footprint" "lasagna-motherboard:ESC" (id 2) (at 238.76 138.43 0)
       (effects (font (size 1.27 1.27)) hide)
     )
@@
     (property "Reference" "U13" (id 0) (at 239.395 144.78 0))
     (property "Value" "ESC" (id 1) (at 239.395 147.32 0))
-    (property "Footprint" "" (id 2) (at 238.76 152.4 0)
+    (property "Footprint" "lasagna-motherboard:ESC" (id 2) (at 238.76 152.4 0)
       (effects (font (size 1.27 1.27)) hide)
     )
@@
     (property "Reference" "U9" (id 0) (at 239.395 90.17 0))
     (property "Value" "ESC" (id 1) (at 239.395 92.71 0))
-    (property "Footprint" "" (id 2) (at 238.76 97.79 0)
+    (property "Footprint" "lasagna-motherboard:ESC" (id 2) (at 238.76 97.79 0)
       (effects (font (size 1.27 1.27)) hide)
     )
@@
     (property "Reference" "U5" (id 0) (at 175.26 58.42 0))
     (property "Value" "Adafruit_PCA9685_PWMGen" (id 1) (at 175.26 60.96 0))
-    (property "Footprint" "" (id 2) (at 194.31 69.85 0)
+    (property "Footprint" "lasagna-motherboard:Adafruit_PCA9685_PWMGen" (id 2) (at 194.31 69.85 0)
       (effects (font (size 1.27 1.27)) hide)
     )
@@
     (property "Reference" "U11" (id 0) (at 239.395 118.11 0))
     (property "Value" "ESC" (id 1) (at 239.395 120.65 0))
-    (property "Footprint" "" (id 2) (at 238.76 125.73 0)
+    (property "Footprint" "lasagna-motherboard:ESC" (id 2) (at 238.76 125.73 0)
       (effects (font (size 1.27 1.27)) hide)
     )
@@
     (property "Reference" "U3" (id 0) (at 103.505 63.5 0))
     (property "Value" "Jetson_Xavier_NX_Pins" (id 1) (at 103.505 66.04 0))
-    (property "Footprint" "" (id 2) (at 93.98 81.28 0)
+    (property "Footprint" "lasagna-motherboard:Jetson_Xavier_NX_2X20_Pin_Header" (id 2) (at 93.98 81.28 0)
       (effects (font (size 1.27 1.27)) hide)
     )
@@
     (property "Reference" "J3" (id 0) (at 243.84 26.67 0))
     (property "Value" "Power_Connector" (id 1) (at 243.84 29.21 0))
-    (property "Footprint" "" (id 2) (at 246.38 33.02 0)
+    (property "Footprint" "lasagna-motherboard:Power_Connector" (id 2) (at 246.38 33.02 0)
       (effects (font (size 1.27 1.27)) hide)
     )
@@
     (property "Reference" "U1" (id 0) (at 40.64 45.72 0))
     (property "Value" "Adafruit_BNO055_IMU" (id 1) (at 33.655 22.86 0))
-    (property "Footprint" "" (id 2) (at 30.48 33.02 0)
+    (property "Footprint" "lasagna-motherboard:Adafruit_BNO055_IMU" (id 2) (at 30.48 33.02 0)
       (effects (font (size 1.27 1.27)) hide)
     )
@@
     (property "Reference" "J2" (id 0) (at 92.71 154.94 0))
     (property "Value" "Fathom_X_Connector" (id 1) (at 92.71 157.48 0))
-    (property "Footprint" "" (id 2) (at 97.79 162.56 0)
+    (property "Footprint" "lasagna-motherboard:FathomX_Connector" (id 2) (at 97.79 162.56 0)
       (effects (font (size 1.27 1.27)) hide)
     )
@@
       (effects (font (size 1.27 1.27)) (justify left))
     )
-    (property "Footprint" "" (id 2) (at 111.76 161.29 0)
+    (property "Footprint" "lasagna-motherboard:FathomX" (id 2) (at 111.76 161.29 0)
       (effects (font (size 1.27 1.27)) hide)
     )
@@
     (property "Reference" "J1" (id 0) (at 52.07 64.77 0))
     (property "Value" "Jetson_Power_Connector" (id 1) (at 52.07 67.31 0))
-    (property "Footprint" "" (id 2) (at 52.07 72.39 0)
+    (property "Footprint" "lasagna-motherboard:Jetson Power Connector" (id 2) (at 52.07 72.39 0)
       (effects (font (size 1.27 1.27)) hide)
     )
@@
     (property "Reference" "U7" (id 0) (at 239.395 55.88 0))
     (property "Value" "ESC" (id 1) (at 239.395 58.42 0))
-    (property "Footprint" "" (id 2) (at 238.76 63.5 0)
+    (property "Footprint" "lasagna-motherboard:ESC" (id 2) (at 238.76 63.5 0)
       (effects (font (size 1.27 1.27)) hide)
     )
@@
     (property "Reference" "U6" (id 0) (at 239.395 41.91 0))
     (property "Value" "ESC" (id 1) (at 239.395 44.45 0))
-    (property "Footprint" "" (id 2) (at 238.76 49.53 0)
+    (property "Footprint" "lasagna-motherboard:ESC" (id 2) (at 238.76 49.53 0)
       (effects (font (size 1.27 1.27)) hide)
     )
@@
     )
     (path "/da79bd2f-f942-4e50-9bea-6468b250780c"
-      (reference "J1") (unit 1) (value "Jetson_Power_Connector") (footprint "")
+      (reference "J1") (unit 1) (value "Jetson_Power_Connector") (footprint "lasagna-motherboard:Jetson Power Connector")
     )
     (path "/ca180f18-8f79-44bf-af5f-17ecc1134053"
-      (reference "J2") (unit 1) (value "Fathom_X_Connector") (footprint "")
+      (reference "J2") (unit 1) (value "Fathom_X_Connector") (footprint "lasagna-motherboard:FathomX_Connector")
     )
     (path "/9b8b9a1b-a1ca-47f4-ab33-f59a78659b22"
-      (reference "J3") (unit 1) (value "Power_Connector") (footprint "")
+      (reference "J3") (unit 1) (value "Power_Connector") (footprint "lasagna-motherboard:Power_Connector")
     )
     (path "/c659a157-8d7b-49bb-b1b7-529e35703d84"
-      (reference "U1") (unit 1) (value "Adafruit_BNO055_IMU") (footprint "")
+      (reference "U1") (unit 1) (value "Adafruit_BNO055_IMU") (footprint "lasagna-motherboard:Adafruit_BNO055_IMU")
     )
     (path "/1f7ea3dc-e040-4340-ac71-367bf56dbd36"
-      (reference "U2") (unit 1) (value "Jetson_Xavier_NX_Mounting_Holes") (footprint "")
+      (reference "U2") (unit 1) (value "Jetson_Xavier_NX_Mounting_Holes") (footprint "lasagna-motherboard:Jetson_Xavier_NX_Mounting_Holes")
     )
     (path "/968fa752-f8dc-4cee-8837-7c67c93064bc"
-      (reference "U3") (unit 1) (value "Jetson_Xavier_NX_Pins") (footprint "")
+      (reference "U3") (unit 1) (value "Jetson_Xavier_NX_Pins") (footprint "lasagna-motherboard:Jetson_Xavier_NX_2X20_Pin_Header")
     )
     (path "/cf27eb86-d6ed-48d5-bd7a-59210dc20ea2"
-      (reference "U4") (unit 1) (value "FathomX") (footprint "")
+      (reference "U4") (unit 1) (value "FathomX") (footprint "lasagna-motherboard:FathomX")
     )
     (path "/77e23894-e0c1-4679-b130-f72b5d52465f"
-      (reference "U5") (unit 1) (value "Adafruit_PCA9685_PWMGen") (footprint "")
+      (reference "U5") (unit 1) (value "Adafruit_PCA9685_PWMGen") (footprint "lasagna-motherboard:Adafruit_PCA9685_PWMGen")
     )
     (path "/e447f43b-8f82-4ceb-87ae-0aec8d2a9782"
-      (reference "U6") (unit 1) (value "ESC") (footprint "")
+      (reference "U6") (unit 1) (value "ESC") (footprint "lasagna-motherboard:ESC")
     )
     (path "/e0af5551-bdbd-4558-bd4f-1d01b5426143"
-      (reference "U7") (unit 1) (value "ESC") (footprint "")
+      (reference "U7") (unit 1) (value "ESC") (footprint "lasagna-motherboard:ESC")
     )
     (path "/1a57f79d-1c0d-41bd-b3e6-e42c42739770"
-      (reference "U8") (unit 1) (value "ESC") (footprint "")
+      (reference "U8") (unit 1) (value "ESC") (footprint "lasagna-motherboard:ESC")
     )
     (path "/73dc5273-435d-4cf1-ba4d-7a495f67c9ba"
-      (reference "U9") (unit 1) (value "ESC") (footprint "")
+      (reference "U9") (unit 1) (value "ESC") (footprint "lasagna-motherboard:ESC")
     )
     (path "/16eb4024-87b6-408d-8ae6-6cc1a1c62ab9"
-      (reference "U10") (unit 1) (value "ESC") (footprint "")
+      (reference "U10") (unit 1) (value "ESC") (footprint "lasagna-motherboard:ESC")
     )
     (path "/8d03dd7c-ed51-4b3a-a5a1-b9fcdd8c7182"
-      (reference "U11") (unit 1) (value "ESC") (footprint "")
+      (reference "U11") (unit 1) (value "ESC") (footprint "lasagna-motherboard:ESC")
     )
     (path "/3615d130-8c2c-45ed-8d95-380df2f08951"
-      (reference "U12") (unit 1) (value "ESC") (footprint "")
+      (reference "U12") (unit 1) (value "ESC") (footprint "lasagna-motherboard:ESC")
     )
     (path "/5431ee3b-1558-45e2-b7d7-b2268d5181fd"
-      (reference "U13") (unit 1) (value "ESC") (footprint "")
-    )
-  )
+      (reference "U13") (unit 1) (value "ESC") (footprint "lasagna-motherboard:ESC")
+    )
+  )

Commit message: created something
Other:
- company: (none) -> Blueshift Robotics
- title: (none) -> Lasagna Motherboard Schematic 
Changed lines of the file:
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@@
 (kicad_sch (version 20211123) (generator eeschema)
   (paper "A4")
+  (title_block
+    (title "Lasagna Motherboard Schematic ")
+    (date "2023-01-03")
+    (rev "v0.1")
+    (company "Blueshift Robotics")
+  )
   (junction (at 77.47 58.42) (diameter 0) (color 0 0 0 0)
   )
