File: lasagna-motherboard/lasagna-motherboard.kicad_sch (KiCad schematic)
At the start: 16 parts, among them J1 Jetson_Power_Connector, J2 Fathom_X_Connector, J3 Power_Connector, U1 Adafruit_BNO055_IMU, U10 ESC, U11 ESC, U12 ESC, U13 ESC, U2 Jetson_Xavier_NX_Mounting_Hol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, U3 Jetson_Xavier_NX_Pins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

Commit message: added the servo connectors
Parts:
- added J? (x2): Servo_Connector, symbol lasagna-motherboard:Servo_Connector
- added U?: ESC_Holder_Mounting_Holes, symbol lasagna-motherboard:ESC_Holder_Mounting_Holes
- added VR? (x2): 7805_TO-220_Voltage_Regulator, symbol lasagna-motherboard:7805_TO-220_Voltage_Regulator
- J1: footprint (none) -> lasagna-motherboard:Jetson Power Connector
- J2: footprint (none) -> lasagna-motherboard:FathomX_Connector
- J3: footprint (none) -> lasagna-motherboard:Power_Connector
- U1: footprint (none) -> lasagna-motherboard:Adafruit_BNO055_IMU
- U10, U11, U12, U13, U6, U7, U8, U9: footprint (none) -> lasagna-motherboard:ESC
- U2: footprint (none) -> lasagna-motherboard:Jetson_Xavier_NX_Mounting_Holes
- U3: footprint (none) -> lasagna-motherboard:Jetson_Xavier_NX_2X20_Pin_Header
- U4: footprint (none) -> lasagna-motherboard:FathomX
- U5: footprint (none) -> lasagna-motherboard:Adafruit_PCA9685_PWMGen
Connections:
- net +12V: now also VR?.1 (VIN), VR?.1 (VIN)
- net +5V: now also J?.2 (VIN), J?.2 (VIN), VR?.3 (VOUT), VR?.3 (VOUT)
- net GND: now also J?.3 (GND), J?.3 (GND), VR?.2 (GND), VR?.2 (GND)
- net at U5.37 (PWM8): now also J?.1 (PWM)
- net at U5.40 (PWM9): now also J?.1 (PWM)
Other:
- company: (none) -> Blueshift Robotics
- title: (none) -> Lasagna Motherboard Schematic 
- moved on the sheet: J2, U4
